File: snowflake2021/snowflake2021.kicad_pcb (KiCad board)
At the start: 2 copper layers, 79 x 86.5 mm, 18 parts, among them J1 AVR-ISP-6, SW1 SW_Push, U1 ATtiny85V-10SU

Commit message: ship it
Parts:
- removed D7: LED, LED_SMD:LED_0603_1608Metric_Pad1.05x0.95mm_HandSolder
- removed the R3 at (142.0, 76.2)
- added D2: LED, LED_SMD:LED_0603_1608Metric_Pad1.05x0.95mm_HandSolder, F.Cu at (173.5, 53.5)
- added R5: 10k, Resistor_SMD:R_1206_3216Metric_Pad1.42x1.75mm_HandSolder, F.Cu at (137.7, 69.8)
- R1: value 10k -> R
- SW1: footprint Button_Switch_THT:SW_PUSH_6mm -> Button_Switch_SMD:SW_Push_1P1T_NO_6x6mm_H9.5mm
- moved D6 63.7 mm to (116.3, 53.2), turned to 60 degrees
- moved D3 57.3 mm to (173.6, 86.4), turned to 240 degrees
- moved J1 39.4 mm to (143.8, 86.4)
- moved D1 30.5 mm to (144.9, 36.8)
- moved SW1 21.8 mm to (144.9, 69.8)
- moved R1 15.1 mm to (156.8, 69.6), turned to 90 degrees
- moved C1 13.3 mm to (135.1, 69.8), turned to 90 degrees
- moved R2 10.9 mm to (146.3, 78.7), turned to 90 degrees
- moved R4 8.90 mm to (154.3, 69.6), turned to 90 degrees
- moved R3 8.15 mm to (143.3, 78.7), turned to 270 degrees
- moved D5 6.77 mm to (116.3, 86.4), turned to 120 degrees
- moved D4 5.08 mm to (144.9, 102.9)
- moved Reset 3.89 mm to (128.0, 57.1), turned to 150 degrees
- moved U1 1.78 mm to (144.9, 60.5)
- renumbered D2 to D1, D8 to D4, D10 to D5, D11 to D6, R4 to R3, R5 to R4, TP1 to Reset
Connections:
- D3 pad 1: row_a -> col_b
- D3 pad 2: col_a -> row_a
- R1 pad 1: VCC -> col_a
- R1 pad 2: rst -> miso
- R2 pad 1: col_a -> col_b
- R2 pad 2: miso -> sck
Routing:
- net row_a: track 42.1 -> 195.8 mm, vias 0 -> 5
- net col_c: track 0.00 -> 64.2 mm, vias 0 -> 3
- net GND: track 0.00 -> 62.1 mm, vias 0 -> 9
- net col_b: track 0.00 -> 54.1 mm, vias 0 -> 2
- net rst: track 0.00 -> 53.1 mm, vias 0 -> 1
- net VCC: track 0.00 -> 50.1 mm
- net sck: track 0.00 -> 47.0 mm, vias 0 -> 1
- net miso: track 0.00 -> 38.3 mm, vias 0 -> 1
- net mosi: track 0.00 -> 37.9 mm, vias 0 -> 1
- net col_a: track 43.3 -> 63.9 mm
- net Net-(R3-Pad1): track 0.00 -> 20.5 mm
- net Net-(SW1-Pad1): track 0.00 -> 6.86 mm
- added copper zone on B.Cu, net GND
- added copper zone on F.Cu, net GND
Other:
- board text added: "+"
- board text added: "-"
- board text added: "JLCJLCJLCJLC"
- board text added: "Merry Christmas! Chris Johnston 2021"
