File: snowflake2021/snowflake2021.sch (KiCad schematic (older format))
At the start: 17 parts, among them J1 AVR-ISP-6, SW1 SW_Push, U1 ATtiny85V-10SU

Commit message: ship it
Parts:
- SW1: footprint Button_Switch_THT:SW_PUSH_6mm -> Button_Switch_SMD:SW_Push_1P1T_NO_6x6mm_H9.5mm
- renumbered D2 to D1, D3 to D2, D7 to D3, D8 to D4, D10 to D5, D11 to D6, R2 to R1, R3 to R2, R4 to R3, R5 to R4, R1 to R5
Changed lines of the file:
@@
 $EndComp
 $Comp
-L power:VCC #PWR0101
+L power:VCC #PWR01
 U 1 1 6188BB86
 P 3000 4150
-F 0 "#PWR0101" H 3000 4000 50  0001 C CNN
+F 0 "#PWR01" H 3000 4000 50  0001 C CNN
 F 1 "VCC" H 3015 4323 50  0000 C CNN
 F 2 "" H 3000 4150 50  0001 C CNN
@@
 $EndComp
 $Comp
-L power:GND #PWR0102
+L power:GND #PWR02
 U 1 1 6188BDE1
 P 3000 4800
-F 0 "#PWR0102" H 3000 4550 50  0001 C CNN
+F 0 "#PWR02" H 3000 4550 50  0001 C CNN
 F 1 "GND" H 3005 4627 50  0000 C CNN
 F 2 "" H 3000 4800 50  0001 C CNN
@@
 	3000 4700 3000 4800
 $Comp
-L power:VCC #PWR0103
+L power:VCC #PWR05
 U 1 1 6188C0EB
 P 3950 3950
-F 0 "#PWR0103" H 3950 3800 50  0001 C CNN
+F 0 "#PWR05" H 3950 3800 50  0001 C CNN
 F 1 "VCC" H 3965 4123 50  0000 C CNN
 F 2 "" H 3950 3950 50  0001 C CNN
@@
 $EndComp
 $Comp
-L power:GND #PWR0104
+L power:GND #PWR06
 U 1 1 6188C435
 P 3950 5200
-F 0 "#PWR0104" H 3950 4950 50  0001 C CNN
+F 0 "#PWR06" H 3950 4950 50  0001 C CNN
 F 1 "GND" H 3955 5027 50  0000 C CNN
 F 2 "" H 3950 5200 50  0001 C CNN
@@
 	3950 4950 3950 5200
 $Comp
-L power:GND #PWR0105
+L power:GND #PWR04
 U 1 1 6188D2B8
 P 3950 3550
-F 0 "#PWR0105" H 3950 3300 50  0001 C CNN
+F 0 "#PWR04" H 3950 3300 50  0001 C CNN
 F 1 "GND" H 3955 3377 50  0000 C CNN
 F 2 "" H 3950 3550 50  0001 C CNN
@@
 $EndComp
 $Comp
-L power:VCC #PWR0106
+L power:VCC #PWR03
 U 1 1 6188D64C
 P 3950 2350
-F 0 "#PWR0106" H 3950 2200 50  0001 C CNN
+F 0 "#PWR03" H 3950 2200 50  0001 C CNN
 F 1 "VCC" H 3965 2523 50  0000 C CNN
 F 2 "" H 3950 2350 50  0001 C CNN
@@
 	4600 3150 4850 3150
 $Comp
-L Device:R R1
+L Device:R R5
 U 1 1 6189837D
 P 5000 3150
-F 0 "R1" V 4793 3150 50  0000 C CNN
+F 0 "R5" V 4793 3150 50  0000 C CNN
 F 1 "10k" V 4884 3150 50  0000 C CNN
 F 2 "Resistor_SMD:R_1206_3216Metric_Pad1.42x1.75mm_HandSolder" V 4930 3150 50  0001 C CNN
@@
 Connection ~ 4850 3150
 $Comp
-L power:VCC #PWR0107
+L power:VCC #PWR07
 U 1 1 61898B8E
 P 5250 3150
-F 0 "#PWR0107" H 5250 3000 50  0001 C CNN
+F 0 "#PWR07" H 5250 3000 50  0001 C CNN
 F 1 "VCC" H 5265 3323 50  0000 C CNN
 F 2 "" H 5250 3150 50  0001 C CNN
@@
 $EndComp
 $Comp
-L power:GND #PWR0108
+L power:GND #PWR08
 U 1 1 61898E34
 P 5250 3550
-F 0 "#PWR0108" H 5250 3300 50  0001 C CNN
+F 0 "#PWR08" H 5250 3300 50  0001 C CNN
 F 1 "GND" H 5255 3377 50  0000 C CNN
 F 2 "" H 5250 3550 50  0001 C CNN
@@
 sck
 $Comp
-L Device:LED D2
+L Device:LED D1
 U 1 1 618F8593
 P 5750 4400
-F 0 "D2" H 5743 4617 50  0000 C CNN
+F 0 "D1" H 5743 4617 50  0000 C CNN
 F 1 "LED" H 5743 4526 50  0000 C CNN
 F 2 "LED_SMD:LED_0603_1608Metric_Pad1.05x0.95mm_HandSolder" H 5750 4400 50  0001 C CNN
@@
 $EndComp
 $Comp
-L Device:LED D7
+L Device:LED D3
 U 1 1 618F8A2C
 P 6200 4400
-F 0 "D7" H 6193 4617 50  0000 C CNN
+F 0 "D3" H 6193 4617 50  0000 C CNN
 F 1 "LED" H 6193 4526 50  0000 C CNN
 F 2 "LED_SMD:LED_0603_1608Metric_Pad1.05x0.95mm_HandSolder" H 6200 4400 50  0001 C CNN
@@
 $EndComp
 $Comp
-L Device:LED D8
+L Device:LED D4
 U 1 1 618F9FF0
 P 6200 4750
-F 0 "D8" H 6193 4967 50  0000 C CNN
+F 0 "D4" H 6193 4967 50  0000 C CNN
 F 1 "LED" H 6193 4876 50  0000 C CNN
 F 2 "LED_SMD:LED_0603_1608Metric_Pad1.05x0.95mm_HandSolder" H 6200 4750 50  0001 C CNN
@@
 $EndComp
 $Comp
-L Device:LED D10
+L Device:LED D5
 U 1 1 618FBE72
 P 6650 4400
-F 0 "D10" H 6643 4617 50  0000 C CNN
+F 0 "D5" H 6643 4617 50  0000 C CNN
 F 1 "LED" H 6643 4526 50  0000 C CNN
 F 2 "LED_SMD:LED_0603_1608Metric_Pad1.05x0.95mm_HandSolder" H 6650 4400 50  0001 C CNN
@@
 $EndComp
 $Comp
-L Device:LED D11
+L Device:LED D6
 U 1 1 618FC275
 P 6650 4750
-F 0 "D11" H 6643 4967 50  0000 C CNN
+F 0 "D6" H 6643 4967 50  0000 C CNN
 F 1 "LED" H 6643 4876 50  0000 C CNN
 F 2 "LED_SMD:LED_0603_1608Metric_Pad1.05x0.95mm_HandSolder" H 6650 4750 50  0001 C CNN
@@
 Connection ~ 3000 4700
 $Comp
-L Device:LED D3
+L Device:LED D2
 U 1 1 618F9B5D
 P 5750 4750
-F 0 "D3" H 5743 4967 50  0000 C CNN
+F 0 "D2" H 5743 4967 50  0000 C CNN
 F 1 "LED" H 5743 4876 50  0000 C CNN
 F 2 "LED_SMD:LED_0603_1608Metric_Pad1.05x0.95mm_HandSolder" H 5750 4750 50  0001 C CNN
@@
 row_a
 $Comp
-L Device:R R2
+L Device:R R1
 U 1 1 6192ECF3
 P 4900 2200
-F 0 "R2" V 4693 2200 50  0000 C CNN
+F 0 "R1" V 4693 2200 50  0000 C CNN
 F 1 "R" V 4784 2200 50  0000 C CNN
 F 2 "Resistor_SMD:R_1206_3216Metric_Pad1.42x1.75mm_HandSolder" V 4830 2200 50  0001 C CNN
@@
 $EndComp
 $Comp
-L Device:R R3
+L Device:R R2
 U 1 1 6192F436
 P 4900 2300
-F 0 "R3" V 4693 2300 50  0000 C CNN
+F 0 "R2" V 4693 2300 50  0000 C CNN
 F 1 "R" V 4784 2300 50  0000 C CNN
 F 2 "Resistor_SMD:R_1206_3216Metric_Pad1.42x1.75mm_HandSolder" V 4830 2300 50  0001 C CNN
@@
 $EndComp
 $Comp
-L Device:R R4
+L Device:R R3
 U 1 1 6192F840
 P 4900 2400
-F 0 "R4" V 5107 2400 50  0000 C CNN
+F 0 "R3" V 5107 2400 50  0000 C CNN
 F 1 "R" V 5016 2400 50  0000 C CNN
 F 2 "Resistor_SMD:R_1206_3216Metric_Pad1.42x1.75mm_HandSolder" V 4830 2400 50  0001 C CNN
@@
 $EndComp
 $Comp
-L Device:R R5
+L Device:R R4
 U 1 1 6192FCB4
 P 4900 2500
-F 0 "R5" V 4693 2500 50  0000 C CNN
+F 0 "R4" V 4693 2500 50  0000 C CNN
 F 1 "R" V 4784 2500 50  0000 C CNN
 F 2 "Resistor_SMD:R_1206_3216Metric_Pad1.42x1.75mm_HandSolder" V 4830 2500 50  0001 C CNN
@@
 F 0 "SW1" H 5750 3335 50  0000 C CNN
 F 1 "SW_Push" H 5750 3244 50  0000 C CNN
-F 2 "Button_Switch_THT:SW_PUSH_6mm" H 5750 3250 50  0001 C CNN
+F 2 "Button_Switch_SMD:SW_Push_1P1T_NO_6x6mm_H9.5mm" H 5750 3250 50  0001 C CNN
 F 3 "~" H 5750 3250 50  0001 C CNN
 	1    5750 3050
@@
 	4550 3050 5550 3050
 $Comp
-L power:GND #PWR0109
+L power:GND #PWR09
 U 1 1 61945365
 P 6100 3050
-F 0 "#PWR0109" H 6100 2800 50  0001 C CNN
+F 0 "#PWR09" H 6100 2800 50  0001 C CNN
 F 1 "GND" H 6105 2877 50  0000 C CNN
 F 2 "" H 6100 3050 50  0001 C CNN
